Commit message: Add Go2 Pinocchio robot model integration

File: go2_description/xacro/leg.xacro (robot description, xacro)
@@ -1,33 +1,37 @@
 <?xml version="1.0"?>
 <robot xmlns:xacro="http://www.ros.org/wiki/xacro">
+  <!--
+    This leg.xacro is aligned with the reference go2_description URDF.
+    Expected macro calls:
+      <xacro:leg name="FL" mirror="1"  mirror_dae="True"  front_hind="1"  front_hind_dae="True"/>
+      <xacro:leg name="FR" mirror="-1" mirror_dae="False" front_hind="1"  front_hind_dae="True"/>
+      <xacro:leg name="RL" mirror="1"  mirror_dae="True"  front_hind="-1" front_hind_dae="False"/>
+      <xacro:leg name="RR" mirror="-1" mirror_dae="False" front_hind="-1" front_hind_dae="False"/>
+    Important:
+      The parent link is base, not trunk.
+  -->
   <xacro:include filename="$(find go2_description)/xacro/transmission.xacro"/>
   <xacro:macro name="leg" params="name mirror mirror_dae front_hind front_hind_dae">
     <joint name="${name}_hip_joint" type="revolute">
-      <xacro:if value="${(mirror_dae == False) and (front_hind_dae == True)}">
-        <origin rpy="0 0 0" xyz="${leg_offset_x} ${-leg_offset_y} 0"/>
-      </xacro:if>
-      <xacro:if value="${(mirror_dae == True) and (front_hind_dae == True)}">
-        <origin rpy="0 0 0" xyz="${leg_offset_x} ${leg_offset_y} 0"/>
-      </xacro:if>
-      <xacro:if value="${(mirror_dae == False) and (front_hind_dae == False)}">
-        <origin rpy="0 0 0" xyz="${-leg_offset_x} ${-leg_offset_y} 0"/>
-      </xacro:if>
-      <xacro:if value="${(mirror_dae == True) and (front_hind_dae == False)}">
-        <origin rpy="0 0 0" xyz="${-leg_offset_x} ${leg_offset_y} 0"/>
-      </xacro:if>
-      <parent link="trunk"/>
+      <origin rpy="0 0 0" xyz="${0.1934 * front_hind} ${0.0465 * mirror} 0"/>
+      <parent link="base"/>
       <child link="${name}_hip"/>
       <axis xyz="1 0 0"/>
-      <dynamics damping="${damping}" friction="${friction}"/>
-      <xacro:if value="${(mirror_dae == True)}">
-        <limit effort="${hip_torque_max}" velocity="${hip_velocity_max}" lower="${hip_position_min}"
-               upper="${hip_position_max}"/>
-      </xacro:if>
-      <xacro:if value="${(mirror_dae == False)}">
-        <limit effort="${hip_torque_max}" velocity="${hip_velocity_max}" lower="${-hip_position_max}"
-               upper="${-hip_position_min}"/>
-      </xacro:if>
+      <limit lower="-1.0472" upper="1.0472" effort="23.7" velocity="30.1"/>
     </joint>
     <link name="${name}_hip">
+      <inertial>
+        <origin
+          xyz="${-0.0054 * front_hind} ${0.00194 * mirror} -0.000105"
+          rpy="0 0 0"/>
+        <mass value="0.678"/>
+        <inertia
+          ixx="0.00048"
+          ixy="${-3.01E-06 * mirror * front_hind}"
+          ixz="${1.11E-06 * front_hind}"
+          iyy="0.000884"
+          iyz="${-1.42E-06 * mirror}"
+          izz="0.000596"/>
+      </inertial>
       <visual>
         <xacro:if value="${(mirror_dae == True) and (front_hind_dae == True)}">
@@ -35,124 +39,188 @@
         </xacro:if>
         <xacro:if value="${(mirror_dae == False) and (front_hind_dae == True)}">
-          <origin rpy="${PI} 0 0" xyz="0 0 0"/>
+          <origin rpy="3.1415 0 0" xyz="0 0 0"/>
         </xacro:if>
         <xacro:if value="${(mirror_dae == True) and (front_hind_dae == False)}">
-          <origin rpy="0 ${PI} 0" xyz="0 0 0"/>
+          <origin rpy="0 3.1415 0" xyz="0 0 0"/>
         </xacro:if>
         <xacro:if value="${(mirror_dae == False) and (front_hind_dae == False)}">
-          <origin rpy="${PI} ${PI} 0" xyz="0 0 0"/>
-        </xacro:if>
-        <geometry>
-          <mesh filename="file://$(find go2_description)/meshes/hip.dae" scale="1 1 1"/>
-        </geometry>
-      </visual>
-      <collision>
-        <origin rpy="${PI/2.0} 0 0" xyz="0 ${hip_offset*mirror} 0"/>
-        <geometry>
-          <cylinder length="${hip_length}" radius="${hip_radius}"/>
-        </geometry>
-      </collision>
-      <inertial>
-        <origin rpy="0 0 0" xyz="${hip_com_x*front_hind} ${hip_com_y*mirror} ${hip_com_z}"/>
-        <mass value="${hip_mass}"/>
-        <inertia
-            ixx="${hip_ixx}" ixy="${hip_ixy*mirror*front_hind}" ixz="${hip_ixz*front_hind}"
-            iyy="${hip_iyy}" iyz="${hip_iyz*mirror}"
-            izz="${hip_izz}"/>
-      </inertial>
+          <origin rpy="3.1415 3.1415 0" xyz="0 0 0"/>
+        </xacro:if>
+        <geometry>
+          <mesh filename="package://go2_description/dae/hip.dae"/>
+        </geometry>
+        <material name="">
+          <color rgba="1 1 1 1"/>
+        </material>
+      </visual>
+      <collision>
+        <origin rpy="1.5707963267948966 0 0" xyz="0 ${0.08 * mirror} 0"/>
+        <geometry>
+          <cylinder length="0.04" radius="0.046"/>
+        </geometry>
+      </collision>
     </link>
     <joint name="${name}_thigh_joint" type="revolute">
-      <origin rpy="0 0 0" xyz="0 ${thigh_offset*mirror} 0"/>
+      <origin rpy="0 0 0" xyz="0 ${0.0955 * mirror} 0"/>
       <parent link="${name}_hip"/>
       <child link="${name}_thigh"/>
       <axis xyz="0 1 0"/>
-      <dynamics damping="${damping}" friction="${friction}"/>
-      <limit effort="${thigh_torque_max}" velocity="${thigh_velocity_max}" lower="${thigh_position_min}"
-             upper="${thigh_position_max}"/>
+      <xacro:if value="${front_hind == 1}">
+        <limit lower="-1.5708" upper="3.4907" effort="23.7" velocity="30.1"/>
+      </xacro:if>
+      <xacro:if value="${front_hind == -1}">
+        <limit lower="-0.5236" upper="4.5379" effort="23.7" velocity="30.1"/>
+      </xacro:if>
     </joint>
     <link name="${name}_thigh">
+      <inertial>
+        <origin
+          xyz="-0.00374 ${-0.0223 * mirror} -0.0327"
+          rpy="0 0 0"/>
+        <mass value="1.152"/>
+        <inertia
+          ixx="0.00584"
+          ixy="${8.72E-05 * mirror}"
+          ixz="-0.000289"
+          iyy="0.0058"
+          iyz="${0.000808 * mirror}"
+          izz="0.00103"/>
+      </inertial>
       <visual>
         <origin rpy="0 0 0" xyz="0 0 0"/>
         <geometry>
           <xacro:if value="${mirror_dae == True}">
-            <mesh filename="file://$(find go2_description)/meshes/thigh.dae" scale="1 1 1"/>
+            <mesh filename="package://go2_description/dae/thigh.dae"/>
           </xacro:if>
           <xacro:if value="${mirror_dae == False}">
-            <mesh filename="file://$(find go2_description)/meshes/thigh_mirror.dae" scale="1 1 1"/>
-          </xacro:if>
-        </geometry>
-      </visual>
-      <collision>
-        <origin rpy="0 ${PI/2.0} 0" xyz="0 0 ${-thigh_length/2.0}"/>
-        <geometry>
-          <box size="${thigh_length} ${thigh_width} ${thigh_height}"/>
-        </geometry>
-      </collision>
-      <inertial>
-        <origin rpy="0 0 0" xyz="${thigh_com_x} ${thigh_com_y*mirror} ${thigh_com_z}"/>
-        <mass value="${thigh_mass}"/>
-        <inertia
-            ixx="${thigh_ixx}" ixy="${thigh_ixy*mirror}" ixz="${thigh_ixz}"
-            iyy="${thigh_iyy}" iyz="${thigh_iyz*mirror}"
-            izz="${thigh_izz}"/>
-      </inertial>
+            <mesh filename="package://go2_description/dae/thigh_mirror.dae"/>
+          </xacro:if>
+        </geometry>
+        <material name="">
+          <color rgba="1 1 1 1"/>
+        </material>
+      </visual>
+      <collision>
+        <origin rpy="0 1.5707963267948966 0" xyz="0 0 -0.1065"/>
+        <geometry>
+          <box size="0.213 0.0245 0.034"/>
+        </geometry>
+      </collision>
     </link>
     <joint name="${name}_calf_joint" type="revolute">
-      <origin rpy="0 0 0" xyz="0 0 ${-thigh_length}"/>
+      <origin rpy="0 0 0" xyz="0 0 -0.213"/>
       <parent link="${name}_thigh"/>
       <child link="${name}_calf"/>
       <axis xyz="0 1 0"/>
-      <dynamics damping="${damping}" friction="${friction}"/>
-      <limit effort="${calf_torque_max}" velocity="${calf_velocity_max}" lower="${calf_position_min}"
-             upper="${calf_position_max}"/>
+      <limit lower="-2.7227" upper="-0.83776" effort="45.43" velocity="15.70"/>
     </joint>
     <link name="${name}_calf">
-      <visual>
-        <origin rpy="0 0 0" xyz="0 0 0"/>
-        <geometry>
-          <mesh filename="file://$(find go2_description)/meshes/calf.dae" scale="1 1 1"/>
-        </geometry>
-      </visual>
-      <collision>
-        <origin rpy="0 ${PI/2.0} 0" xyz="0 0 ${-calf_length/2.0}"/>
-        <geometry>
-          <box size="${calf_length} ${calf_width} ${calf_height}"/>
-        </geometry>
-      </collision>
-      <inertial>
-        <origin rpy="0 0 0" xyz="${calf_com_x} ${calf_com_y} ${calf_com_z}"/>
-        <mass value="${calf_mass}"/>
-        <inertia
-            ixx="${calf_ixx}" ixy="${calf_ixy}" ixz="${calf_ixz}"
-            iyy="${calf_iyy}" iyz="${calf_iyz}"
-            izz="${calf_izz}"/>
-      </inertial>
-    </link>
-    <joint name="${name}_foot_fixed" type="fixed">
-      <origin rpy="0 0 0" xyz="0 0 ${-(calf_length)}"/>
+      <inertial>
+        <origin
+          xyz="0.00548 ${-0.000975 * mirror} -0.115"
+          rpy="0 0 0"/>
+        <mass value="0.154"/>
+        <inertia
+          ixx="0.00108"
+          ixy="${3.4E-07 * mirror}"
+          ixz="1.72E-05"
+          iyy="0.0011"
+          iyz="${8.28E-06 * mirror}"
+          izz="3.29E-05"/>
+      </inertial>
+      <visual>
+        <origin rpy="0 0 0" xyz="0 0 0"/>
+        <geometry>
+          <xacro:if value="${mirror_dae == True}">
+            <mesh filename="package://go2_description/dae/calf.dae"/>
+          </xacro:if>
+          <xacro:if value="${mirror_dae == False}">
+            <mesh filename="package://go2_description/dae/calf_mirror.dae"/>
+          </xacro:if>
+        </geometry>
+        <material name="">
+          <color rgba="1 1 1 1"/>
+        </material>
+      </visual>
+      <!-- Reference URDF uses slightly different calf collision for FL. -->
+      <xacro:if value="${name == 'FL'}">
+        <collision>
+          <origin rpy="0 -0.21 0" xyz="0.008 0 -0.06"/>
+          <geometry>
+            <cylinder length="0.12" radius="0.012"/>
+          </geometry>
+        </collision>
+      </xacro:if>
+      <xacro:unless value="${name == 'FL'}">
+        <collision>
+          <origin rpy="0 -0.2 0" xyz="0.01 0 -0.06"/>
+          <geometry>
+            <cylinder length="0.12" radius="0.013"/>
+          </geometry>
+        </collision>
+      </xacro:unless>
+    </link>
+    <link name="${name}_calflower">
+      <collision>
+        <origin rpy="0 0 0" xyz="0 0 0"/>
+        <geometry>
+          <cylinder length="0.065" radius="0.011"/>
+        </geometry>
+      </collision>
+    </link>
+    <joint name="${name}_calflower_joint" type="fixed">
+      <origin xyz="0.020 0 -0.148" rpy="0 0.05 0"/>
+      <parent link="${name}_calf"/>
+      <child link="${name}_calflower"/>
+      <axis xyz="0 0 0"/>
+    </joint>
+    <link name="${name}_calflower1">
+      <collision>
+        <origin rpy="0 0 0" xyz="0 0 0"/>
+        <geometry>
+          <cylinder length="0.03" radius="0.0155"/>
+        </geometry>
+      </collision>
+    </link>
+    <joint name="${name}_calflower1_joint" type="fixed">
+      <origin xyz="-0.01 0 -0.04" rpy="0 0.48 0"/>
+      <parent link="${name}_calflower"/>
+      <child link="${name}_calflower1"/>
+      <axis xyz="0 0 0"/>
+    </joint>
+    <link name="${name}_foot">
+      <inertial>
+        <origin xyz="0 0 0" rpy="0 0 0"/>
+        <mass value="0.04"/>
+        <inertia
+          ixx="9.6e-06"
+          ixy="0"
+          ixz="0"
+          iyy="9.6e-06"
+          iyz="0"
+          izz="9.6e-06"/>
+      </inertial>
+      <visual>
+        <origin xyz="0 0 0" rpy="0 0 0"/>
+        <geometry>
+          <mesh filename="package://go2_description/dae/foot.dae"/>
+        </geometry>
+        <material name="">
+          <color rgba="1 1 1 1"/>
+        </material>
+      </visual>
+      <collision>
+        <origin rpy="0 0 0" xyz="-0.002 0 0"/>
+        <geometry>
+          <sphere radius="0.022"/>
+        </geometry>
+      </collision>
+    </link>
+    <joint name="${name}_foot_joint" type="fixed" dont_collapse="true">
+      <origin xyz="0 0 -0.213" rpy="0 0 0"/>
       <parent link="${name}_calf"/>
       <child link="${name}_foot"/>
-    </joint>
-    <link name="${name}_foot">
-      <visual>
-        <origin rpy="0 0 0" xyz="0 0 0"/>
-        <geometry>
-          <sphere radius="${foot_radius-0.01}"/>
-        </geometry>
-      </visual>
-      <collision>
-        <origin rpy="0 0 0" xyz="0 0 0"/>
-        <geometry>
-          <sphere radius="${foot_radius}"/>
-        </geometry>
-      </collision>
-      <inertial>
-        <mass value="${foot_mass}"/>
-        <inertia
-            ixx="${(2*foot_mass)/5.0*(foot_radius*foot_radius)}" ixy="0.0" ixz="0.0"
-            iyy="${(2*foot_mass)/5.0*(foot_radius*foot_radius)}" iyz="0.0"
-            izz="${(2*foot_mass)/5.0*(foot_radius*foot_radius)}"/>
-      </inertial>
-    </link>
+      <axis xyz="0 0 0"/>
+    </joint>
     <gazebo reference="${name}_hip">
       <mu1>0.2</mu1>

File: go2_description/xacro/robot.xacro (robot description, xacro)
@@ -23,110 +23,126 @@
   <!-- Actually, the rotor will rotate and the joint is not fixed. Reduction ratio should be considered. -->
   <!-- Debug mode will hung up the robot, use "true" or "false" to switch it. -->
-  <xacro:if value="$(arg DEBUG)">
-    <link name="world"/>
-    <joint name="base_static_joint" type="fixed">
-      <origin rpy="0 0 0" xyz="0 0 0"/>
-      <parent link="world"/>
-      <child link="base"/>
-    </joint>
-  </xacro:if>
+  <!-- ========================= -->
+  <!-- Base body                 -->
+  <!-- ========================= -->
   <link name="base">
+    <inertial>
+      <origin xyz="0.021112 0 -0.005366" rpy="0 0 0"/>
+      <mass value="6.921"/>
+      <inertia
+        ixx="0.02448"
+        ixy="0.00012166"
+        ixz="0.0014849"
+        iyy="0.098077"
+        iyz="-3.12E-05"
+        izz="0.107"/>
+    </inertial>
     <visual>
-      <origin rpy="0 0 0" xyz="0 0 0"/>
+      <origin xyz="0 0 0" rpy="0 0 0"/>
       <geometry>
-        <box size="0.001 0.001 0.001"/>
+        <mesh filename="package://go2_description/dae/base.dae"/>
       </geometry>
-    </visual>
-  </link>
-  <joint name="floating_base" type="fixed">
-    <origin rpy="0 0 0" xyz="0 0 0"/>
-    <parent link="base"/>
-    <child link="trunk"/>
-  </joint>
-  <link name="trunk">
-    <visual>
-      <origin rpy="0 0 0" xyz="0 0 0"/>
-      <geometry>
-        <mesh filename="file://$(find go2_description)/meshes/trunk.dae" scale="1 1 1"/>
-      </geometry>
-      <!-- <material name="orange"/> -->
+      <material name="base_white">
+        <color rgba="1 1 1 1"/>
+      </material>
     </visual>
     <collision>
-      <origin rpy="0 0 0" xyz="0 0 0"/>
+      <origin xyz="0 0 0" rpy="0 0 0"/>
       <geometry>
-        <box size="${trunk_length} ${trunk_width} ${trunk_height}"/>
+        <box size="0.3762 0.0935 0.114"/>
       </geometry>
     </collision>
+  </link>
+<link name="Head_upper">
+    <inertial>
+      <origin xyz="0 0 0" rpy="0 0 0"/>
+      <mass value="0.001"/>
+      <inertia
+        ixx="9.6e-06"
+        ixy="0"
+        ixz="0"
+        iyy="9.6e-06"
+        iyz="0"
+        izz="9.6e-06"/>
+    </inertial>
     <collision>
-      <origin rpy="0 0 0" xyz="0 0 0"/>
+      <origin xyz="0 0 0" rpy="0 0 0"/>
       <geometry>
-        <box size="0.1881 0.04675 0.057"/>
+        <cylinder radius="0.05" length="0.09"/>
       </geometry>
     </collision>
+  </link>
+  <joint name="Head_upper_joint" type="fixed" dont_collapse="true">
+    <origin xyz="0.285 0 0.01" rpy="0 0 0"/>
+    <parent link="base"/>
+    <child link="Head_upper"/>
+    <axis xyz="0 0 0"/>
+  </joint>
+  <link name="Head_lower">
+    <inertial>
+      <origin xyz="0 0 0" rpy="0 0 0"/>
+      <mass value="0.001"/>
+      <inertia
+        ixx="9.6e-06"
+        ixy="0"
+        ixz="0"
+        iyy="9.6e-06"
+        iyz="0"
+        izz="9.6e-06"/>
+    </inertial>
     <collision>
-      <origin rpy="0 0 0" xyz="0.285 0 0.01"/>
+      <origin xyz="0 0 0" rpy="0 0 0"/>
       <geometry>
-        <cylinder length="0.05" radius="0.045"/>
+        <sphere radius="0.047"/>
       </geometry>
     </collision>
-    <collision>
-      <origin rpy="0 0 0" xyz="0.293 0 -0.06"/>
-      <geometry>
-        <box size="0.047 0.047 0.047"/>
-      </geometry>
-    </collision>
+  </link>
+  <joint name="Head_lower_joint" type="fixed" dont_collapse="true">
+    <origin xyz="0.008 0 -0.07" rpy="0 0 0"/>
+    <parent link="Head_upper"/>
+    <child link="Head_lower"/>
+    <axis xyz="0 0 0"/>
+  </joint>
+  <link name="imu">
     <inertial>
-      <origin rpy="0 0 0" xyz="${trunk_com_x} ${trunk_com_y} ${trunk_com_z}"/>
-      <mass value="${trunk_mass}"/>
+      <origin xyz="0 0 0" rpy="0 0 0"/>
+      <mass value="0"/>
       <inertia
-          ixx="${trunk_ixx}" ixy="${trunk_ixy}" ixz="${trunk_ixz}"
-          iyy="${trunk_iyy}" iyz="${trunk_iyz}"
-          izz="${trunk_izz}"/>
+        ixx="0"
+        ixy="0"
+        ixz="0"
+        iyy="0"
+        iyz="0"
+        izz="0"/>
     </inertial>
   </link>
   <joint name="imu_joint" type="fixed">
-    <parent link="trunk"/>
-    <child link="imu_link"/>
-    <origin rpy="0 0 0" xyz="0 0 0"/>
-  </joint>
-  <link name="imu_link">
-    <inertial>
-      <mass value="0.001"/>
-      <origin rpy="0 0 0" xyz="0 0 0"/>
-      <inertia ixx="0.0001" ixy="0" ixz="0" iyy="0.0001" iyz="0" izz="0.0001"/>
-    </inertial>
-    <visual>
-      <origin rpy="0 0 0" xyz="0 0 0"/>
-      <geometry>
-        <box size="0.001 0.001 0.001"/>
-      </geometry>
-      <!-- <material name="red"/> -->
-    </visual>
-    <collision>
-      <origin rpy="0 0 0" xyz="0 0 0"/>
-      <geometry>
-        <box size=".001 .001 .001"/>
-      </geometry>
-    </collision>
-  </link>
-  <joint name="camera_joint_front" type="fixed">
-    <parent link="trunk"/>
-    <child link="front_camera"/>
-    <origin rpy="0 0 0" xyz="0.32715 0 0.04297"/>
-  </joint>
-  <link name="front_camera">
-  </link>
-  <joint name="lidar_joint" type="fixed">
-    <origin
-        xyz="0.28945 0 -0.046825" rpy="0 2.8782 0"/>
-    <parent link="trunk"/>
-    <child link="lidar"/>
+    <origin xyz="-0.02557 0 0.04232" rpy="0 0 0"/>
+    <parent link="base"/>
+    <child link="imu"/>
     <axis xyz="0 0 0"/>
   </joint>
-  <link name="lidar">
+  <link name="radar">
+    <inertial>
+      <origin xyz="0 0 0" rpy="0 0 0"/>
+      <mass value="0"/>
+      <inertia
+        ixx="0"
+        ixy="0"
+        ixz="0"
+        iyy="0"
+        iyz="0"
+        izz="0"/>
+    </inertial>
   </link>
-  <xacro:leg name="FR" mirror="-1" mirror_dae="False" front_hind="1" front_hind_dae="True"/>
-  <xacro:leg name="FL" mirror="1" mirror_dae="True" front_hind="1" front_hind_dae="True"/>
+  <joint name="radar_joint" type="fixed">
+    <origin xyz="0.28945 0 -0.046825" rpy="0 2.8782 0"/>
+    <parent link="base"/>
+    <child link="radar"/>
+    <axis xyz="0 0 0"/>
+  </joint>
+  <xacro:leg name="FL" mirror="1"  mirror_dae="True"  front_hind="1"  front_hind_dae="True"/>
+  <xacro:leg name="FR" mirror="-1" mirror_dae="False" front_hind="1"  front_hind_dae="True"/>
+  <xacro:leg name="RL" mirror="1"  mirror_dae="True"  front_hind="-1" front_hind_dae="False"/>
   <xacro:leg name="RR" mirror="-1" mirror_dae="False" front_hind="-1" front_hind_dae="False"/>
-  <xacro:leg name="RL" mirror="1" mirror_dae="True" front_hind="-1" front_hind_dae="False"/>
 </robot>

File: go2_description/xacro/ros2_control.xacro (robot description, xacro)
@@ -10,4 +10,34 @@
   			<param name="viewer_refresh_hz">60.0</param>
 			</hardware>
+		<joint name="FL_hip_joint">
+			<command_interface name="position"/>
+			<command_interface name="velocity"/>
+			<command_interface name="effort"/>
+			<command_interface name="kp"/>
+			<command_interface name="kd"/>
+			<state_interface name="position"/>
+			<state_interface name="velocity"/>
+			<state_interface name="effort"/>
+		</joint>
+		<joint name="FL_thigh_joint">
+			<command_interface name="position"/>
+			<command_interface name="velocity"/>
+			<command_interface name="effort"/>
+			<command_interface name="kp"/>
+			<command_interface name="kd"/>
+			<state_interface name="position"/>
+			<state_interface name="velocity"/>
+			<state_interface name="effort"/>
+		</joint>
+		<joint name="FL_calf_joint">
+			<command_interface name="position"/>
+			<command_interface name="velocity"/>
+			<command_interface name="effort"/>
+			<command_interface name="kp"/>
+			<command_interface name="kd"/>
+			<state_interface name="position"/>
+			<state_interface name="velocity"/>
+			<state_interface name="effort"/>
+		</joint>
 		<joint name="FR_hip_joint">
 			<command_interface name="position"/>
@@ -40,5 +70,5 @@
 			<state_interface name="effort"/>
 		</joint>
-		<joint name="FL_hip_joint">
+		<joint name="RL_hip_joint">
 			<command_interface name="position"/>
 			<command_interface name="velocity"/>
@@ -50,5 +80,5 @@
 			<state_interface name="effort"/>
 		</joint>
-		<joint name="FL_thigh_joint">
+		<joint name="RL_thigh_joint">
 			<command_interface name="position"/>
 			<command_interface name="velocity"/>
@@ -60,5 +90,5 @@
 			<state_interface name="effort"/>
 		</joint>
-		<joint name="FL_calf_joint">
+		<joint name="RL_calf_joint">
 			<command_interface name="position"/>
 			<command_interface name="velocity"/>
@@ -100,34 +130,4 @@
 			<state_interface name="effort"/>
 		</joint>
-		<joint name="RL_hip_joint">
-			<command_interface name="position"/>
-			<command_interface name="velocity"/>
-			<command_interface name="effort"/>
-			<command_interface name="kp"/>
-			<command_interface name="kd"/>
-			<state_interface name="position"/>
-			<state_interface name="velocity"/>
-			<state_interface name="effort"/>
-		</joint>
-		<joint name="RL_thigh_joint">
-			<command_interface name="position"/>
-			<command_interface name="velocity"/>
-			<command_interface name="effort"/>
-			<command_interface name="kp"/>
-			<command_interface name="kd"/>
-			<state_interface name="position"/>
-			<state_interface name="velocity"/>
-			<state_interface name="effort"/>
-		</joint>
-		<joint name="RL_calf_joint">
-			<command_interface name="position"/>
-			<command_interface name="velocity"/>
-			<command_interface name="effort"/>
-			<command_interface name="kp"/>
-			<command_interface name="kd"/>
-			<state_interface name="position"/>
-			<state_interface name="velocity"/>
-			<state_interface name="effort"/>
-		</joint>
 		<sensor name="imu_sensor">
 			<state_interface name="orientation.w"/>
